Commit message: feat: 更新LHandPro模型文件并修改相关配置
更新了LHandPro的STL模型文件，添加了新的DH116S-R000-A1.urdf模型描述文件
移除了旧的DH126S模型文件，修改了package.xml和setup.py中的描述信息
更新了README.md中的项目标题和启动命令，调整了CANFD初始化代码

File: src/lhandpro_description/urdf/DH116S-R000-A1.urdf (robot description, URDF)
Before this commit: robot DH126S-L000-A1, 17 links, 16 joints
Links:
- removed link finger11_Link
- removed link finger12_Link
- removed link finger13_Link
- removed link finger14_Link
- removed link finger21_Link
- removed link finger22_Link
- removed link finger23_Link
- removed link finger31_Link
- removed link finger32_Link
- removed link finger33_Link
- removed link finger41_Link
- removed link finger42_Link
- removed link finger43_Link
- removed link finger51_Link
- removed link finger52_Link
- removed link finger53_Link
- added link finger11_link, mass 0.0027298; collision mesh filename=package://lhandpro_description/meshes/finger11_link.STL; visual mesh filename=package://lhandpro_description/meshes/finger11_link.STL
- added link finger12_link, mass 0.15691; collision mesh filename=package://lhandpro_description/meshes/finger12_link.STL; visual mesh filename=package://lhandpro_description/meshes/finger12_link.STL
- added link finger13_link, mass 0.0051235; collision mesh filename=package://lhandpro_description/meshes/finger13_link.STL; visual mesh filename=package://lhandpro_description/meshes/finger13_link.STL
- added link finger14_link, mass 0.0024048; collision mesh filename=package://lhandpro_description/meshes/finger14_link.STL; visual mesh filename=package://lhandpro_description/meshes/finger14_link.STL
- added link finger21_link, mass 0.0039377; collision mesh filename=package://lhandpro_description/meshes/finger21_link.STL; visual mesh filename=package://lhandpro_description/meshes/finger21_link.STL
- added link finger22_link, mass 0.0035951; collision mesh filename=package://lhandpro_description/meshes/finger22_link.STL; visual mesh filename=package://lhandpro_description/meshes/finger22_link.STL
- added link finger23_link, mass 0.0019493; collision mesh filename=package://lhandpro_description/meshes/finger23_link.STL; visual mesh filename=package://lhandpro_description/meshes/finger23_link.STL
- added link finger31_link, mass 0.0046564; collision mesh filename=package://lhandpro_description/meshes/finger31_link.STL; visual mesh filename=package://lhandpro_description/meshes/finger31_link.STL
- added link finger32_link, mass 0.0039648; collision mesh filename=package://lhandpro_description/meshes/finger32_link.STL; visual mesh filename=package://lhandpro_description/meshes/finger32_link.STL
- added link finger33_link, mass 0.0022727; collision mesh filename=package://lhandpro_description/meshes/finger33_link.STL; visual mesh filename=package://lhandpro_description/meshes/finger33_link.STL
- added link finger41_link, mass 0.0041427; collision mesh filename=package://lhandpro_description/meshes/finger41_link.STL; visual mesh filename=package://lhandpro_description/meshes/finger41_link.STL
- added link finger42_link, mass 0.0038285; collision mesh filename=package://lhandpro_description/meshes/finger42_link.STL; visual mesh filename=package://lhandpro_description/meshes/finger42_link.STL
- added link finger43_link, mass 0.0019493; collision mesh filename=package://lhandpro_description/meshes/finger43_link.STL; visual mesh filename=package://lhandpro_description/meshes/finger43_link.STL
- added link finger51_link, mass 0.0034504; collision mesh filename=package://lhandpro_description/meshes/finger51_link.STL; visual mesh filename=package://lhandpro_description/meshes/finger51_link.STL
- added link finger52_link, mass 0.0034587; collision mesh filename=package://lhandpro_description/meshes/finger52_link.STL; visual mesh filename=package://lhandpro_description/meshes/finger52_link.STL
- added link finger53_link, mass 0.0014968; collision mesh filename=package://lhandpro_description/meshes/finger53_link.STL; visual mesh filename=package://lhandpro_description/meshes/finger53_link.STL
- link base_link: mass 0.11674 -> 0.10795
Joints:
- joint finger11: axis 0 0 1 -> 0 0 -1; child finger11_Link -> finger11_link; limit lower=-1.57 upper=1.57 effort=0 velocity=0 -> lower=0 upper=1.92 effort=0 velocity=0; origin xyz=0.018 -0.021464 0.040041 rpy=0.087266 0 0 -> xyz=0.019011 -0.007805 0.03432 rpy=0 -3.0438E-05 1.5708
- joint finger12: axis 0 -1 0 -> -1 0 0; child finger12_Link -> finger12_link; origin xyz=0.018876 -0.0049375 -0.0023593 rpy=0 0.95149 -0.25585 -> xyz=-0.0024172 -0.015 0.0067143 rpy=1.1997 -0.2618 0; parent finger11_Link -> finger11_link
- joint finger13: axis 0 -1 0 -> -1 0 0; child finger13_Link -> finger13_link; origin xyz=0 0 0.045 rpy=0 0 0 -> xyz=0 0 0.040273 rpy=0 0 0; parent finger12_Link -> finger12_link
- joint finger14: child finger14_Link -> finger14_link; limit lower=0 upper=1.57 effort=0 velocity=0 -> lower=0 upper=0 effort=0 velocity=0; parent finger13_Link -> finger13_link
- joint finger21: axis 0 1 0 -> 1 0 0; child finger21_Link -> finger21_link; origin xyz=-0.011581 -0.031971 0.10003 rpy=0.052657 0.10625 0.0055894 -> xyz=0.026269 0.0052799 0.083877 rpy=-0.018831 0.11816 -0.15867
- joint finger22: axis 0 1 0 -> 1 0 0; child finger22_Link -> finger22_link; origin xyz=0 0 0.035 rpy=0 0 0 -> xyz=0 -0.0036408 0.027789 rpy=0 0 0; parent finger21_Link -> finger21_link
- joint finger23: child finger23_Link -> finger23_link; limit lower=0 upper=1.57 effort=0 velocity=0 -> lower=0 upper=0 effort=0 velocity=0; parent finger22_Link -> finger22_link
- joint finger31: axis 0 1 0 -> 1 0 0; child finger31_Link -> finger31_link; origin xyz=-0.013501 -0.0105 0.10286 rpy=0 0.10214 0 -> xyz=0.008744 0.006507 0.088166 rpy=0.10576 0.052052 -0.049525
- joint finger32: axis 0 1 0 -> 1 0 0; child finger32_Link -> finger32_link; origin xyz=0 0 0.035 rpy=0 0 0 -> xyz=0 -0.00026526 0.03253 rpy=0 0 0; parent finger31_Link -> finger31_link
- joint finger33: child finger33_Link -> finger33_link; limit lower=0 upper=1.57 effort=0 velocity=0 -> lower=0 upper=0 effort=0 velocity=0; parent finger32_Link -> finger32_link
- joint finger41: axis 0 1 0 -> 1 0 0; child finger41_Link -> finger41_link; origin xyz=-0.015081 0.010971 0.10183 rpy=-0.052889 0.14148 -0.0074648 -> xyz=-0.0088463 0.0073041 0.087413 rpy=0.082606 -0.034779 0.050937
- joint finger42: axis 0 1 0 -> 1 0 0; child finger42_Link -> finger42_link; origin xyz=0 0 0.035 rpy=0 0 0 -> xyz=0 0 0.029529 rpy=-0.084349 0 0; parent finger41_Link -> finger41_link
- joint finger43: child finger43_Link -> finger43_link; limit lower=0 upper=1.57 effort=0 velocity=0 -> lower=0 upper=0 effort=0 velocity=0; parent finger42_Link -> finger42_link
- joint finger51: axis 0 1 0 -> 1 0 0; child finger51_Link -> finger51_link; origin xyz=-0.013081 0.032156 0.097798 rpy=-0.078754 0.073706 -0.0058113 -> xyz=-0.026313 0.0056254 0.083042 rpy=0.076915 -0.11667 0.14928
- joint finger52: axis 0 1 0 -> 1 0 0; child finger52_Link -> finger52_link; origin xyz=0 0 0.035 rpy=0 0 0 -> xyz=0 0 0.025024 rpy=0 0 0; parent finger51_Link -> finger51_link
- joint finger53: child finger53_Link -> finger53_link; limit lower=0 upper=1.57 effort=0 velocity=0 -> (none); parent finger52_Link -> finger52_link
