Commit message: refactor(urdf): 更新mesh文件路径至lhandpro_description包

File: src/lhandpro_description/urdf/DH116-L000-A1.urdf (robot description, URDF)
Before this commit: robot DH116-L000-A1, 17 links, 16 joints
Links:
- link base_link: geometry collision mesh filename=package://lhandpro_description/meshes/base_link.STL; visual mesh filename=package://lhandpro_description/meshes/base_link.STL
- link finger11_Link: geometry collision mesh filename=package://lhandpro_description/meshes/finger11_Link.STL; visual mesh filename=package://lhandpro_description/meshes/finger11_Link.STL
- link finger12_Link: geometry collision mesh filename=package://lhandpro_description/meshes/finger12_Link.STL; visual mesh filename=package://lhandpro_description/meshes/finger12_Link.STL
- link finger13_Link: geometry collision mesh filename=package://lhandpro_description/meshes/finger13_Link.STL; visual mesh filename=package://lhandpro_description/meshes/finger13_Link.STL
- link finger14_Link: geometry collision mesh filename=package://lhandpro_description/meshes/finger14_Link.STL; visual mesh filename=package://lhandpro_description/meshes/finger14_Link.STL
- link finger21_Link: geometry collision mesh filename=package://lhandpro_description/meshes/finger21_Link.STL; visual mesh filename=package://lhandpro_description/meshes/finger21_Link.STL
- link finger22_Link: geometry collision mesh filename=package://lhandpro_description/meshes/finger22_Link.STL; visual mesh filename=package://lhandpro_description/meshes/finger22_Link.STL
- link finger23_Link: geometry collision mesh filename=package://lhandpro_description/meshes/finger23_Link.STL; visual mesh filename=package://lhandpro_description/meshes/finger23_Link.STL
- link finger31_Link: geometry collision mesh filename=package://lhandpro_description/meshes/finger31_Link.STL; visual mesh filename=package://lhandpro_description/meshes/finger31_Link.STL
- link finger32_Link: geometry collision mesh filename=package://lhandpro_description/meshes/finger32_Link.STL; visual mesh filename=package://lhandpro_description/meshes/finger32_Link.STL
- link finger33_Link: geometry collision mesh filename=package://lhandpro_description/meshes/finger33_Link.STL; visual mesh filename=package://lhandpro_description/meshes/finger33_Link.STL
- link finger41_Link: geometry collision mesh filename=package://lhandpro_description/meshes/finger41_Link.STL; visual mesh filename=package://lhandpro_description/meshes/finger41_Link.STL
- link finger42_Link: geometry collision mesh filename=package://lhandpro_description/meshes/finger42_Link.STL; visual mesh filename=package://lhandpro_description/meshes/finger42_Link.STL
- link finger43_Link: geometry collision mesh filename=package://lhandpro_description/meshes/finger43_Link.STL; visual mesh filename=package://lhandpro_description/meshes/finger43_Link.STL
- link finger51_Link: geometry collision mesh filename=package://lhandpro_description/meshes/finger51_Link.STL; visual mesh filename=package://lhandpro_description/meshes/finger51_Link.STL
- link finger52_Link: geometry collision mesh filename=package://lhandpro_description/meshes/finger52_Link.STL; visual mesh filename=package://lhandpro_description/meshes/finger52_Link.STL
- link finger53_Link: geometry collision mesh filename=package://lhandpro_description/meshes/finger53_Link.STL; visual mesh filename=package://lhandpro_description/meshes/finger53_Link.STL

File: src/lhandpro_description/urdf/DH116-R000-A1.urdf (robot description, URDF)
Before this commit: robot DH116-R000-A1, 17 links, 16 joints
Links:
- link base_link: geometry collision mesh filename=package://lhandpro_description/meshes/base_link.STL; visual mesh filename=package://lhandpro_description/meshes/base_link.STL
- link finger11_link: geometry collision mesh filename=package://lhandpro_description/meshes/finger11_link.STL; visual mesh filename=package://lhandpro_description/meshes/finger11_link.STL
- link finger12_link: geometry collision mesh filename=package://lhandpro_description/meshes/finger12_link.STL; visual mesh filename=package://lhandpro_description/meshes/finger12_link.STL
- link finger13_link: geometry collision mesh filename=package://lhandpro_description/meshes/finger13_link.STL; visual mesh filename=package://lhandpro_description/meshes/finger13_link.STL
- link finger14_link: geometry collision mesh filename=package://lhandpro_description/meshes/finger14_link.STL; visual mesh filename=package://lhandpro_description/meshes/finger14_link.STL
- link finger21_link: geometry collision mesh filename=package://lhandpro_description/meshes/finger21_link.STL; visual mesh filename=package://lhandpro_description/meshes/finger21_link.STL
- link finger22_link: geometry collision mesh filename=package://lhandpro_description/meshes/finger22_link.STL; visual mesh filename=package://lhandpro_description/meshes/finger22_link.STL
- link finger23_link: geometry collision mesh filename=package://lhandpro_description/meshes/finger23_link.STL; visual mesh filename=package://lhandpro_description/meshes/finger23_link.STL
- link finger31_link: geometry collision mesh filename=package://lhandpro_description/meshes/finger31_link.STL; visual mesh filename=package://lhandpro_description/meshes/finger31_link.STL
- link finger32_link: geometry collision mesh filename=package://lhandpro_description/meshes/finger32_link.STL; visual mesh filename=package://lhandpro_description/meshes/finger32_link.STL
- link finger33_link: geometry collision mesh filename=package://lhandpro_description/meshes/finger33_link.STL; visual mesh filename=package://lhandpro_description/meshes/finger33_link.STL
- link finger41_link: geometry collision mesh filename=package://lhandpro_description/meshes/finger41_link.STL; visual mesh filename=package://lhandpro_description/meshes/finger41_link.STL
- link finger42_link: geometry collision mesh filename=package://lhandpro_description/meshes/finger42_link.STL; visual mesh filename=package://lhandpro_description/meshes/finger42_link.STL
- link finger43_link: geometry collision mesh filename=package://lhandpro_description/meshes/finger43_link.STL; visual mesh filename=package://lhandpro_description/meshes/finger43_link.STL
- link finger51_link: geometry collision mesh filename=package://lhandpro_description/meshes/finger51_link.STL; visual mesh filename=package://lhandpro_description/meshes/finger51_link.STL
- link finger52_link: geometry collision mesh filename=package://lhandpro_description/meshes/finger52_link.STL; visual mesh filename=package://lhandpro_description/meshes/finger52_link.STL
- link finger53_link: geometry collision mesh filename=package://lhandpro_description/meshes/finger53_link.STL; visual mesh filename=package://lhandpro_description/meshes/finger53_link.STL
